Commit message: fix: base_hand, orca_hand, robotis_hx5_d20 URDF 메시 경로 수정

File: base_hand/urdf/left.urdf (robot description, URDF)
Before this commit: robot left_hand, 28 links, 27 joints
Links:
- link left_index_dip: geometry visual mesh filename=package://atlas_hand/models/base_hand/meshes/left/index_dip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 scale=0.1 0.1 0.1
- link left_index_mcp: geometry visual mesh filename=package://atlas_hand/models/base_hand/meshes/left/index_mcp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 scale=0.1 0.1 0.1
- link left_index_pip: geometry visual mesh filename=package://atlas_hand/models/base_hand/meshes/left/index_pip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 scale=0.1 0.1 0.1
- link left_middle_dip: geometry visual mesh filename=package://atlas_hand/models/base_hand/meshes/left/middle_di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 scale=0.1 0.1 0.1
- link left_middle_mcp: geometry visual mesh filename=package://atlas_hand/models/base_hand/meshes/left/middle_mc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 scale=0.1 0.1 0.1
- link left_middle_pip: geometry visual mesh filename=package://atlas_hand/models/base_hand/meshes/left/middle_pi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 scale=0.1 0.1 0.1
- link left_pinky_dip: geometry visual mesh filename=package://atlas_hand/models/base_hand/meshes/left/pinky_dip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 scale=0.1 0.1 0.1
- link left_pinky_mcp: geometry visual mesh filename=package://atlas_hand/models/base_hand/meshes/left/pinky_mcp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 scale=0.1 0.1 0.1
- link left_pinky_pip: geometry visual mesh filename=package://atlas_hand/models/base_hand/meshes/left/pinky_pip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 scale=0.1 0.1 0.1
- link left_ring_dip: geometry visual mesh filename=package://atlas_hand/models/base_hand/meshes/left/ring_dip.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 scale=0.1 0.1 0.1
- link left_ring_mcp: geometry visual mesh filename=package://atlas_hand/models/base_hand/meshes/left/ring_mcp.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 scale=0.1 0.1 0.1
- link left_ring_pip: geometry visual mesh filename=package://atlas_hand/models/base_hand/meshes/left/ring_pip.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 scale=0.1 0.1 0.1
- link left_thumb_cmc0: geometry visual mesh filename=package://atlas_hand/models/base_hand/meshes/left/thumb_cmc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 scale=0.1 0.1 0.1
- link left_thumb_cmc1: geometry visual mesh filename=package://atlas_hand/models/base_hand/meshes/left/thumb_cmc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 scale=0.1 0.1 0.1
- link left_thumb_ip: geometry visual mesh filename=package://atlas_hand/models/base_hand/meshes/left/thumb_ip.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 scale=0.1 0.1 0.1
- link left_thumb_mcp: geometry visual mesh filename=package://atlas_hand/models/base_hand/meshes/left/thumb_mcp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 scale=0.1 0.1 0.1
- link left_wrist: geometry visual mesh filename=package://atlas_hand/models/base_hand/meshes/left/wrist_lef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 scale=0.1 0.1 0.1

File: base_hand/urdf/right.urdf (robot description, URDF)
Before this commit: robot right_hand, 28 links, 27 joints
Links:
- link right_index_dip: geometry visual mesh filename=package://atlas_hand/models/base_hand/meshes/right/index_di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 scale=0.1 0.1 0.1
- link right_index_mcp: geometry visual mesh filename=package://atlas_hand/models/base_hand/meshes/right/index_mc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 scale=0.1 0.1 0.1
- link right_index_pip: geometry visual mesh filename=package://atlas_hand/models/base_hand/meshes/right/index_pi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 scale=0.1 0.1 0.1
- link right_middle_dip: geometry visual mesh filename=package://atlas_hand/models/base_hand/meshes/right/middle_d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 scale=0.1 0.1 0.1
- link right_middle_mcp: geometry visual mesh filename=package://atlas_hand/models/base_hand/meshes/right/middle_m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 scale=0.1 0.1 0.1
- link right_middle_pip: geometry visual mesh filename=package://atlas_hand/models/base_hand/meshes/right/middle_p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 scale=0.1 0.1 0.1
- link right_pinky_dip: geometry visual mesh filename=package://atlas_hand/models/base_hand/meshes/right/pinky_di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 scale=0.1 0.1 0.1
- link right_pinky_mcp: geometry visual mesh filename=package://atlas_hand/models/base_hand/meshes/right/pinky_mc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 scale=0.1 0.1 0.1
- link right_pinky_pip: geometry visual mesh filename=package://atlas_hand/models/base_hand/meshes/right/pinky_pi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 scale=0.1 0.1 0.1
- link right_ring_dip: geometry visual mesh filename=package://atlas_hand/models/base_hand/meshes/right/ring_dip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 scale=0.1 0.1 0.1
- link right_ring_mcp: geometry visual mesh filename=package://atlas_hand/models/base_hand/meshes/right/ring_mcp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 scale=0.1 0.1 0.1
- link right_ring_pip: geometry visual mesh filename=package://atlas_hand/models/base_hand/meshes/right/ring_pip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 scale=0.1 0.1 0.1
- link right_thumb_cmc0: geometry visual mesh filename=package://atlas_hand/models/base_hand/meshes/right/thumb_cm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 scale=0.1 0.1 0.1
- link right_thumb_cmc1: geometry visual mesh filename=package://atlas_hand/models/base_hand/meshes/right/thumb_cm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 scale=0.1 0.1 0.1
- link right_thumb_ip: geometry visual mesh filename=package://atlas_hand/models/base_hand/meshes/right/thumb_ip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 scale=0.1 0.1 0.1
- link right_thumb_mcp: geometry visual mesh filename=package://atlas_hand/models/base_hand/meshes/right/thumb_mc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 scale=0.1 0.1 0.1
- link right_wrist: geometry visual mesh filename=package://atlas_hand/models/base_hand/meshes/right/wrist_ri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 scale=0.1 0.1 0.1

File: orca_hand/urdf/left.urdf (robot description, URDF)
Before this commit: robot orcahand_left, 19 links, 18 joints
Links:
- link ForeArmStructure-Model_e18f2368: geometry visual mesh filename=package://atlas_hand/models/orca_hand/meshes/left/ForeArmSt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 scale=0.001 0.001 0.001
- link I-AP-L_57ce92f7: geometry visual mesh filename=package://atlas_hand/models/orca_hand/meshes/left/I-AP-L.stl scale=0.001 0.001 0.001
- link I-FingerTipAssembly_ed91b18a: geometry visual mesh filename=package://atlas_hand/models/orca_hand/meshes/left/I-FingerT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 scale=0.001 0.001 0.001
- link I-PP_3df4f91d: geometry visual mesh filename=package://atlas_hand/models/orca_hand/meshes/left/I-PP.stl scale=0.001 0.001 0.001
- link L-Carpals_719fff8c: geometry visual mesh filename=package://atlas_hand/models/orca_hand/meshes/left/L-Carpals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 scale=0.001 0.001 0.001
- link L-T-AP_58680c44: geometry visual mesh filename=package://atlas_hand/models/orca_hand/meshes/left/L-T-AP.stl scale=0.001 0.001 0.001
- link M-AP_6ec59111: geometry visual mesh filename=package://atlas_hand/models/orca_hand/meshes/left/M-AP.stl scale=0.001 0.001 0.001
- link M-AP_e04a96f2: geometry visual mesh filename=package://atlas_hand/models/orca_hand/meshes/left/M-AP.stl scale=0.001 0.001 0.001
- link M-FingerTipAssembly_34afb748: geometry visual mesh filename=package://atlas_hand/models/orca_hand/meshes/left/M-FingerT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 scale=0.001 0.001 0.001
- link M-FingerTipAssembly_424a8e75: geometry visual mesh filename=package://atlas_hand/models/orca_hand/meshes/left/M-FingerT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 scale=0.001 0.001 0.001
- link M-PP_08efa608: geometry visual mesh filename=package://atlas_hand/models/orca_hand/meshes/left/M-PP.stl scale=0.001 0.001 0.001
- link M-PP_8660a1eb: geometry visual mesh filename=package://atlas_hand/models/orca_hand/meshes/left/M-PP.stl scale=0.001 0.001 0.001
- link P-AP_f5e42b61: geometry visual mesh filename=package://atlas_hand/models/orca_hand/meshes/left/P-AP.stl scale=0.001 0.001 0.001
- link P-FingerTipAssembly_cd219176: geometry visual mesh filename=package://atlas_hand/models/orca_hand/meshes/left/P-FingerT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 scale=0.001 0.001 0.001
- link P-PP_1d411b9b: geometry visual mesh filename=package://atlas_hand/models/orca_hand/meshes/left/P-PP.stl scale=0.001 0.001 0.001
- link T-DP_307db3cc: geometry visual mesh filename=package://atlas_hand/models/orca_hand/meshes/left/T-DP.stl scale=0.001 0.001 0.001
- link T-PP_ef067304: geometry visual mesh filename=package://atlas_hand/models/orca_hand/meshes/left/T-PP.stl scale=0.001 0.001 0.001
- link T-TP-L_92b8100b: geometry visual mesh filename=package://atlas_hand/models/orca_hand/meshes/left/T-TP-L.stl scale=0.001 0.001 0.001
- link TopTower-Model_4a80d30e: geometry visual mesh filename=package://atlas_hand/models/orca_hand/meshes/left/TopTower-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 scale=0.001 0.001 0.001

File: orca_hand/urdf/right.urdf (robot description, URDF)
Before this commit: robot orcahand_right, 24 links, 23 joints
Links:
- link ForeArmStructure-Model_e18f2368: geometry visual mesh filename=package://atlas_hand/models/orca_hand/meshes/right/ForeArmS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 scale=0.001 0.001 0.001
- link I-AP-R_d95d02d1: geometry visual mesh filename=package://atlas_hand/models/orca_hand/meshes/right/I-AP-R.s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 scale=0.001 0.001 0.001
- link I-FingerTipAssembly_ec49c16c: geometry visual mesh filename=package://atlas_hand/models/orca_hand/meshes/right/I-Finger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 scale=0.001 0.001 0.001
- link I-PP_bacbd481: geometry visual mesh filename=package://atlas_hand/models/orca_hand/meshes/right/I-PP.stl scale=0.001 0.001 0.001
- link M-AP_6ec59111: geometry visual mesh filename=package://atlas_hand/models/orca_hand/meshes/right/M-AP.stl scale=0.001 0.001 0.001
- link M-AP_e04a96f2: geometry visual mesh filename=package://atlas_hand/models/orca_hand/meshes/right/M-AP.stl scale=0.001 0.001 0.001
- link M-FingerTipAssembly_34afb748: geometry visual mesh filename=package://atlas_hand/models/orca_hand/meshes/right/M-Finger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 scale=0.001 0.001 0.001
- link M-FingerTipAssembly_424a8e75: geometry visual mesh filename=package://atlas_hand/models/orca_hand/meshes/right/M-Finger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 scale=0.001 0.001 0.001
- link M-PP_08efa608: geometry visual mesh filename=package://atlas_hand/models/orca_hand/meshes/right/M-PP.stl scale=0.001 0.001 0.001
- link M-PP_8660a1eb: geometry visual mesh filename=package://atlas_hand/models/orca_hand/meshes/right/M-PP.stl scale=0.001 0.001 0.001
- link P-AP_f5e42b61: geometry visual mesh filename=package://atlas_hand/models/orca_hand/meshes/right/P-AP.stl scale=0.001 0.001 0.001
- link P-FingerTipAssembly_cd219176: geometry visual mesh filename=package://atlas_hand/models/orca_hand/meshes/right/P-Finger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 scale=0.001 0.001 0.001
- link P-PP_1d411b9b: geometry visual mesh filename=package://atlas_hand/models/orca_hand/meshes/right/P-PP.stl scale=0.001 0.001 0.001
- link R-Carpals_8d1f1041: geometry visual mesh filename=package://atlas_hand/models/orca_hand/meshes/right/R-Carpal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 scale=0.001 0.001 0.001
- link R-T-AP_a9723101: geometry visual mesh filename=package://atlas_hand/models/orca_hand/meshes/right/R-T-AP.s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 scale=0.001 0.001 0.001
- link T-DP_b7429e50: geometry visual mesh filename=package://atlas_hand/models/orca_hand/meshes/right/T-DP.stl scale=0.001 0.001 0.001
- link T-PP_68395e98: geometry visual mesh filename=package://atlas_hand/models/orca_hand/meshes/right/T-PP.stl scale=0.001 0.001 0.001
- link T-TP-R_1c2b802d: geometry visual mesh filename=package://atlas_hand/models/orca_hand/meshes/right/T-TP-R.s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 scale=0.001 0.001 0.001
- link TopTower-Model_4a80d30e: geometry visual mesh filename=package://atlas_hand/models/orca_hand/meshes/right/TopTower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 scale=0.001 0.001 0.001

File: robotis_hx5_d20/urdf/hx5_d20_left.urdf (robot description, URDF)
Before this commit: robot hand_generated, 26 links, 25 joints
Links:
- link finger_l_link1: geometry collision mesh filename=package://atlas_hand/models/robotis_hx5_d20/meshes/hx5_d20_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 scale=0.001 0.001 0.001; visual mesh filename=package://atlas_hand/models/robotis_hx5_d20/meshes/hx5_d20_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 scale=0.001 0.001 0.001
- link finger_l_link10: geometry collision mesh filename=package://atlas_hand/models/robotis_hx5_d20/meshes/hx5_d20_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 scale=0.001 0.001 0.001; visual mesh filename=package://atlas_hand/models/robotis_hx5_d20/meshes/hx5_d20_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 scale=0.001 0.001 0.001
- link finger_l_link11: geometry collision mesh filename=package://atlas_hand/models/robotis_hx5_d20/meshes/hx5_d20_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 scale=0.001 0.001 0.001; visual mesh filename=package://atlas_hand/models/robotis_hx5_d20/meshes/hx5_d20_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 scale=0.001 0.001 0.001
- link finger_l_link12: geometry collision mesh filename=package://atlas_hand/models/robotis_hx5_d20/meshes/hx5_d20_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 scale=0.001 0.001 0.001; visual mesh filename=package://atlas_hand/models/robotis_hx5_d20/meshes/hx5_d20_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 scale=0.001 0.001 0.001
- link finger_l_link13: geometry collision mesh filename=package://atlas_hand/models/robotis_hx5_d20/meshes/hx5_d20_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 scale=0.001 0.001 0.001; visual mesh filename=package://atlas_hand/models/robotis_hx5_d20/meshes/hx5_d20_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 scale=0.001 0.001 0.001
- link finger_l_link14: geometry collision mesh filename=package://atlas_hand/models/robotis_hx5_d20/meshes/hx5_d20_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 scale=0.001 0.001 0.001; visual mesh filename=package://atlas_hand/models/robotis_hx5_d20/meshes/hx5_d20_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 scale=0.001 0.001 0.001
- link finger_l_link15: geometry collision mesh filename=package://atlas_hand/models/robotis_hx5_d20/meshes/hx5_d20_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 scale=0.001 0.001 0.001; visual mesh filename=package://atlas_hand/models/robotis_hx5_d20/meshes/hx5_d20_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 scale=0.001 0.001 0.001
- link finger_l_link16: geometry collision mesh filename=package://atlas_hand/models/robotis_hx5_d20/meshes/hx5_d20_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 scale=0.001 0.001 0.001; visual mesh filename=package://atlas_hand/models/robotis_hx5_d20/meshes/hx5_d20_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 scale=0.001 0.001 0.001
- link finger_l_link17: geometry collision mesh filename=package://atlas_hand/models/robotis_hx5_d20/meshes/hx5_d20_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 scale=0.001 0.001 0.001; visual mesh filename=package://atlas_hand/models/robotis_hx5_d20/meshes/hx5_d20_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 scale=0.001 0.001 0.001
- link finger_l_link18: geometry collision mesh filename=package://atlas_hand/models/robotis_hx5_d20/meshes/hx5_d20_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 scale=0.001 0.001 0.001; visual mesh filename=package://atlas_hand/models/robotis_hx5_d20/meshes/hx5_d20_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 scale=0.001 0.001 0.001
- link finger_l_link19: geometry collision mesh filename=package://atlas_hand/models/robotis_hx5_d20/meshes/hx5_d20_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 scale=0.001 0.001 0.001; visual mesh filename=package://atlas_hand/models/robotis_hx5_d20/meshes/hx5_d20_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 scale=0.001 0.001 0.001
- link finger_l_link2: geometry collision mesh filename=package://atlas_hand/models/robotis_hx5_d20/meshes/hx5_d20_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 scale=0.001 0.001 0.001; visual mesh filename=package://atlas_hand/models/robotis_hx5_d20/meshes/hx5_d20_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 scale=0.001 0.001 0.001
- link finger_l_link20: geometry collision mesh filename=package://atlas_hand/models/robotis_hx5_d20/meshes/hx5_d20_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 scale=0.001 0.001 0.001; visual mesh filename=package://atlas_hand/models/robotis_hx5_d20/meshes/hx5_d20_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 scale=0.001 0.001 0.001
- link finger_l_link3: geometry collision mesh filename=package://atlas_hand/models/robotis_hx5_d20/meshes/hx5_d20_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 scale=0.001 0.001 0.001; visual mesh filename=package://atlas_hand/models/robotis_hx5_d20/meshes/hx5_d20_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 scale=0.001 0.001 0.001
- link finger_l_link4: geometry collision mesh filename=package://atlas_hand/models/robotis_hx5_d20/meshes/hx5_d20_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 scale=0.001 0.001 0.001; visual mesh filename=package://atlas_hand/models/robotis_hx5_d20/meshes/hx5_d20_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 scale=0.001 0.001 0.001
- link finger_l_link5: geometry collision mesh filename=package://atlas_hand/models/robotis_hx5_d20/meshes/hx5_d20_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 scale=0.001 0.001 0.001; visual mesh filename=package://atlas_hand/models/robotis_hx5_d20/meshes/hx5_d20_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 scale=0.001 0.001 0.001
- link finger_l_link6: geometry collision mesh filename=package://atlas_hand/models/robotis_hx5_d20/meshes/hx5_d20_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 scale=0.001 0.001 0.001; visual mesh filename=package://atlas_hand/models/robotis_hx5_d20/meshes/hx5_d20_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 scale=0.001 0.001 0.001
- link finger_l_link7: geometry collision mesh filename=package://atlas_hand/models/robotis_hx5_d20/meshes/hx5_d20_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 scale=0.001 0.001 0.001; visual mesh filename=package://atlas_hand/models/robotis_hx5_d20/meshes/hx5_d20_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 scale=0.001 0.001 0.001
- link finger_l_link8: geometry collision mesh filename=package://atlas_hand/models/robotis_hx5_d20/meshes/hx5_d20_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 scale=0.001 0.001 0.001; visual mesh filename=package://atlas_hand/models/robotis_hx5_d20/meshes/hx5_d20_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 scale=0.001 0.001 0.001
- link finger_l_link9: geometry collision mesh filename=package://atlas_hand/models/robotis_hx5_d20/meshes/hx5_d20_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 scale=0.001 0.001 0.001; visual mesh filename=package://atlas_hand/models/robotis_hx5_d20/meshes/hx5_d20_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 scale=0.001 0.001 0.001
- link hx5_d20_left_base: geometry collision mesh filename=package://atlas_hand/models/robotis_hx5_d20/meshes/hx5_d20_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 scale=0.001 0.001 0.001; visual mesh filename=package://atlas_hand/models/robotis_hx5_d20/meshes/hx5_d20_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 scale=0.001 0.001 0.001

File: robotis_hx5_d20/urdf/hx5_d20_right.urdf (robot description, URDF)
Before this commit: robot hand_generated, 26 links, 25 joints
Links:
- link finger_r_link1: geometry collision mesh filename=package://atlas_hand/models/robotis_hx5_d20/meshes/hx5_d20_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 scale=0.001 0.001 0.001; visual mesh filename=package://atlas_hand/models/robotis_hx5_d20/meshes/hx5_d20_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 scale=0.001 0.001 0.001
- link finger_r_link10: geometry collision mesh filename=package://atlas_hand/models/robotis_hx5_d20/meshes/hx5_d20_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 scale=0.001 0.001 0.001; visual mesh filename=package://atlas_hand/models/robotis_hx5_d20/meshes/hx5_d20_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 scale=0.001 0.001 0.001
- link finger_r_link11: geometry collision mesh filename=package://atlas_hand/models/robotis_hx5_d20/meshes/hx5_d20_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 scale=0.001 0.001 0.001; visual mesh filename=package://atlas_hand/models/robotis_hx5_d20/meshes/hx5_d20_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 scale=0.001 0.001 0.001
- link finger_r_link12: geometry collision mesh filename=package://atlas_hand/models/robotis_hx5_d20/meshes/hx5_d20_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 scale=0.001 0.001 0.001; visual mesh filename=package://atlas_hand/models/robotis_hx5_d20/meshes/hx5_d20_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 scale=0.001 0.001 0.001
- link finger_r_link13: geometry collision mesh filename=package://atlas_hand/models/robotis_hx5_d20/meshes/hx5_d20_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 scale=0.001 0.001 0.001; visual mesh filename=package://atlas_hand/models/robotis_hx5_d20/meshes/hx5_d20_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 scale=0.001 0.001 0.001
- link finger_r_link14: geometry collision mesh filename=package://atlas_hand/models/robotis_hx5_d20/meshes/hx5_d20_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 scale=0.001 0.001 0.001; visual mesh filename=package://atlas_hand/models/robotis_hx5_d20/meshes/hx5_d20_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 scale=0.001 0.001 0.001
- link finger_r_link15: geometry collision mesh filename=package://atlas_hand/models/robotis_hx5_d20/meshes/hx5_d20_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 scale=0.001 0.001 0.001; visual mesh filename=package://atlas_hand/models/robotis_hx5_d20/meshes/hx5_d20_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 scale=0.001 0.001 0.001
- link finger_r_link16: geometry collision mesh filename=package://atlas_hand/models/robotis_hx5_d20/meshes/hx5_d20_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 scale=0.001 0.001 0.001; visual mesh filename=package://atlas_hand/models/robotis_hx5_d20/meshes/hx5_d20_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 scale=0.001 0.001 0.001
- link finger_r_link17: geometry collision mesh filename=package://atlas_hand/models/robotis_hx5_d20/meshes/hx5_d20_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 scale=0.001 0.001 0.001; visual mesh filename=package://atlas_hand/models/robotis_hx5_d20/meshes/hx5_d20_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 scale=0.001 0.001 0.001
- link finger_r_link18: geometry collision mesh filename=package://atlas_hand/models/robotis_hx5_d20/meshes/hx5_d20_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 scale=0.001 0.001 0.001; visual mesh filename=package://atlas_hand/models/robotis_hx5_d20/meshes/hx5_d20_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 scale=0.001 0.001 0.001
- link finger_r_link19: geometry collision mesh filename=package://atlas_hand/models/robotis_hx5_d20/meshes/hx5_d20_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 scale=0.001 0.001 0.001; visual mesh filename=package://atlas_hand/models/robotis_hx5_d20/meshes/hx5_d20_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 scale=0.001 0.001 0.001
- link finger_r_link2: geometry collision mesh filename=package://atlas_hand/models/robotis_hx5_d20/meshes/hx5_d20_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 scale=0.001 0.001 0.001; visual mesh filename=package://atlas_hand/models/robotis_hx5_d20/meshes/hx5_d20_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 scale=0.001 0.001 0.001
- link finger_r_link20: geometry collision mesh filename=package://atlas_hand/models/robotis_hx5_d20/meshes/hx5_d20_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 scale=0.001 0.001 0.001; visual mesh filename=package://atlas_hand/models/robotis_hx5_d20/meshes/hx5_d20_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 scale=0.001 0.001 0.001
- link finger_r_link3: geometry collision mesh filename=package://atlas_hand/models/robotis_hx5_d20/meshes/hx5_d20_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 scale=0.001 0.001 0.001; visual mesh filename=package://atlas_hand/models/robotis_hx5_d20/meshes/hx5_d20_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 scale=0.001 0.001 0.001
- link finger_r_link4: geometry collision mesh filename=package://atlas_hand/models/robotis_hx5_d20/meshes/hx5_d20_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 scale=0.001 0.001 0.001; visual mesh filename=package://atlas_hand/models/robotis_hx5_d20/meshes/hx5_d20_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 scale=0.001 0.001 0.001
- link finger_r_link5: geometry collision mesh filename=package://atlas_hand/models/robotis_hx5_d20/meshes/hx5_d20_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 scale=0.001 0.001 0.001; visual mesh filename=package://atlas_hand/models/robotis_hx5_d20/meshes/hx5_d20_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 scale=0.001 0.001 0.001
- link finger_r_link6: geometry collision mesh filename=package://atlas_hand/models/robotis_hx5_d20/meshes/hx5_d20_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 scale=0.001 0.001 0.001; visual mesh filename=package://atlas_hand/models/robotis_hx5_d20/meshes/hx5_d20_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 scale=0.001 0.001 0.001
- link finger_r_link7: geometry collision mesh filename=package://atlas_hand/models/robotis_hx5_d20/meshes/hx5_d20_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 scale=0.001 0.001 0.001; visual mesh filename=package://atlas_hand/models/robotis_hx5_d20/meshes/hx5_d20_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 scale=0.001 0.001 0.001
- link finger_r_link8: geometry collision mesh filename=package://atlas_hand/models/robotis_hx5_d20/meshes/hx5_d20_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 scale=0.001 0.001 0.001; visual mesh filename=package://atlas_hand/models/robotis_hx5_d20/meshes/hx5_d20_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 scale=0.001 0.001 0.001
- link finger_r_link9: geometry collision mesh filename=package://atlas_hand/models/robotis_hx5_d20/meshes/hx5_d20_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 scale=0.001 0.001 0.001; visual mesh filename=package://atlas_hand/models/robotis_hx5_d20/meshes/hx5_d20_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 scale=0.001 0.001 0.001
- link hx5_d20_right_base: geometry collision mesh filename=package://atlas_hand/models/robotis_hx5_d20/meshes/hx5_d20_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 scale=0.001 0.001 0.001; visual mesh filename=package://atlas_hand/models/robotis_hx5_d20/meshes/hx5_d20_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 scale=0.001 0.001 0.001
