Commit message: fix: orca hand 링크 관성·질량 메시 기반 재계산 (SolidWorks 단위오류 교정)
orca hand URDF의 inertial 19개 링크 전부가 계통적 단위오류로 관성이 물리적
불가능값이었음(예: ForeArmStructure mass 7.4kg·I=132kg·m² → 반경 4m 필요).
이 오염이 소비자(dex_vla USD / dex_mj MJCF)에서 손목 유효관성을 137kg·m²로
부풀려 팔 제어 발산·궤적 불일치를 유발.

각 링크 STL(스케일 0.001, mm→m)에서 부피·COM·관성텐서를 계산해:
- 관성: <inertial><origin>=메시 COM, <inertia>=COM 기준 전체 텐서로 재기입.
- 질량: 손 전체를 균일 플라스틱 밀도(1100kg/m³)로 재계산(팁 과중·ForeArm
  강철급 질량이 contact 물리를 왜곡했으므로). 손 총질량 ~7.7kg→1.63kg.
right/left 양쪽 적용.

Co-Authored-By: Claude Opus 4.8 <noreply@anthropic.com>
Claude-Session: https://claude.ai/code/session_01Ex6DscjiRkBfpMWq18tqtX

File: dexhand_description/orca_hand/urdf/left.urdf (robot description, URDF)
Before this commit: robot orcahand_left, 19 links, 18 joints
Links:
- link ForeArmStructure-Model_e18f2368: mass 7.422534035794272 -> 1.03986168
- link I-AP-L_57ce92f7: mass 0.004581542163025142 -> 0.00420410837
- link I-FingerTipAssembly_ed91b18a: mass 0.04675178908397048 -> 0.0132619276
- link I-PP_3df4f91d: mass 0.011373207304546197 -> 0.0164134871
- link L-Carpals_719fff8c: mass 0.8542565487567293 -> 0.199928939
- link L-T-AP_58680c44: mass 0.007005325272888604 -> 0.00673926605
- link M-AP_6ec59111: mass 0.004923565158859135 -> 0.00457455603
- link M-AP_e04a96f2: mass 0.004923565158859135 -> 0.00457455603
- link M-FingerTipAssembly_34afb748: mass 0.04673701376980013 -> 0.0132619276
- link M-FingerTipAssembly_424a8e75: mass 0.04673701376980013 -> 0.0132619276
- link M-PP_08efa608: mass 0.012733573971304512 -> 0.0180811266
- link M-PP_8660a1eb: mass 0.012733573971304512 -> 0.0180811266
- link P-AP_f5e42b61: mass 0.004135862855401387 -> 0.00372082918
- link P-FingerTipAssembly_cd219176: mass 0.033190557637887204 -> 0.00969327969
- link P-PP_1d411b9b: mass 0.008117379921259958 -> 0.0120334203
- link T-DP_307db3cc: mass 0.00815768733004441 -> 0.0093098726
- link T-PP_ef067304: mass 0.010490827160908196 -> 0.0155568868
- link T-TP-L_92b8100b: mass 0.007979567574495501 -> 0.0170557923
- link TopTower-Model_4a80d30e: mass 0.18565193224536478 -> 0.201151391

File: dexhand_description/orca_hand/urdf/right.urdf (robot description, URDF)
Before this commit: robot orcahand_right, 24 links, 23 joints
Links:
- link ForeArmStructure-Model_e18f2368: mass 7.422534035794272 -> 1.03986168
- link I-AP-R_d95d02d1: mass 0.004590288233037025 -> 0.00421344458
- link I-FingerTipAssembly_ec49c16c: mass 0.04675178908397048 -> 0.0132619276
- link I-PP_bacbd481: mass 0.011373207304546197 -> 0.0164134871
- link M-AP_6ec59111: mass 0.004923565158859135 -> 0.00457455603
- link M-AP_e04a96f2: mass 0.004923565158859135 -> 0.00457455603
- link M-FingerTipAssembly_34afb748: mass 0.04673701376980013 -> 0.0132619276
- link M-FingerTipAssembly_424a8e75: mass 0.04673701376980013 -> 0.0132619276
- link M-PP_08efa608: mass 0.012733573971304512 -> 0.0180811266
- link M-PP_8660a1eb: mass 0.012733573971304512 -> 0.0180811266
- link P-AP_f5e42b61: mass 0.004135862855401387 -> 0.00372082918
- link P-FingerTipAssembly_cd219176: mass 0.033190557637887204 -> 0.00969327969
- link P-PP_1d411b9b: mass 0.008117379921259958 -> 0.0120334203
- link R-Carpals_8d1f1041: mass 0.13538810897856451 -> 0.205723302
- link R-T-AP_a9723101: mass 0.007004136465100992 -> 0.00673510435
- link T-DP_b7429e50: mass 0.00815768733004441 -> 0.0093098726
- link T-PP_68395e98: mass 0.010490827160908196 -> 0.0155568868
- link T-TP-R_1c2b802d: mass 0.00797873207561227 -> 0.01705578
- link TopTower-Model_4a80d30e: mass 0.18565193224536478 -> 0.201151391

Commit message: feat(orca_hand): add tactile sensor frames to left/right URDFs
Downstream consumers derive the real-hardware finger→joint mapping from
sensor frames (`{side}_sensor_dorsum` + `{side}_sensor_{finger}_{proximal,distal}`).
Without them whatslab-sdk cannot map ORCA hand joints and falls back to an
error, so users had to point WHATSLAB_MODELS_ROOT at an out-of-tree copy.

Additive only: 11 links + 11 joints per side, appended before </robot>.
No existing link, joint, origin, axis or limit is touched.

Verified on both sides:
  - XML parses; pinocchio builds the model, nq = 17 (unchanged)
  - all six required sensor frames exist as BODY frames
  - finger→joint mapping resolves: thumb 6, index/middle/ring/pinky 5 each

Co-Authored-By: Claude Opus 5 <noreply@anthropic.com>

File: dexhand_description/orca_hand/urdf/left.urdf (robot description, URDF)
Before this commit: robot orcahand_left, 19 links, 18 joints
Links:
- added link left_sensor_dorsum
- added link left_sensor_index_distal
- added link left_sensor_index_proximal
- added link left_sensor_middle_distal
- added link left_sensor_middle_proximal
- added link left_sensor_pinky_distal
- added link left_sensor_pinky_proximal
- added link left_sensor_ring_distal
- added link left_sensor_ring_proximal
- added link left_sensor_thumb_distal
- added link left_sensor_thumb_proximal
Joints:
- added joint left_sensor_dorsum_fixed: type fixed, parent L-Carpals_719fff8c, child left_sensor_dorsum, origin xyz=0 0 0 rpy=1.57 0 0
- added joint left_sensor_index_distal_fixed: type fixed, parent I-FingerTipAssembly_ed91b18a, child left_sensor_index_distal, origin xyz=-0.004946 0.000001 0.045049 rpy=1.00 0 1.57
- added joint left_sensor_index_proximal_fixed: type fixed, parent I-PP_3df4f91d, child left_sensor_index_proximal, origin xyz=0.00075 0 0.0185 rpy=1.00 0 1.57
- added joint left_sensor_middle_distal_fixed: type fixed, parent M-FingerTipAssembly_34afb748, child left_sensor_middle_distal, origin xyz=-0.004946 0.000001 0.045049 rpy=1.00 0 1.57
- added joint left_sensor_middle_proximal_fixed: type fixed, parent M-PP_08efa608, child left_sensor_middle_proximal, origin xyz=0.001 0 0.02 rpy=1.00 0 1.57
- added joint left_sensor_pinky_distal_fixed: type fixed, parent P-FingerTipAssembly_cd219176, child left_sensor_pinky_distal, origin xyz=-0.005452 0.000005 0.038056 rpy=1.00 0 1.57
- added joint left_sensor_pinky_proximal_fixed: type fixed, parent P-PP_1d411b9b, child left_sensor_pinky_proximal, origin xyz=0.0005 0 0.0155 rpy=1.00 0 1.57
- added joint left_sensor_ring_distal_fixed: type fixed, parent M-FingerTipAssembly_424a8e75, child left_sensor_ring_distal, origin xyz=-0.004946 0.000001 0.045049 rpy=1.00 0 1.57
- added joint left_sensor_ring_proximal_fixed: type fixed, parent M-PP_8660a1eb, child left_sensor_ring_proximal, origin xyz=0.001 0 0.02 rpy=1.00 0 1.57
- added joint left_sensor_thumb_distal_fixed: type fixed, parent T-DP_307db3cc, child left_sensor_thumb_distal, origin xyz=0.004104 -0.00019 0.030238 rpy=1.57 0 1.57
- added joint left_sensor_thumb_proximal_fixed: type fixed, parent T-PP_ef067304, child left_sensor_thumb_proximal, origin xyz=0.0005 0 0.016 rpy=1.57 0 1.57

File: dexhand_description/orca_hand/urdf/right.urdf (robot description, URDF)
Before this commit: robot orcahand_right, 24 links, 23 joints
Links:
- added link right_sensor_dorsum
- added link right_sensor_index_distal
- added link right_sensor_index_proximal
- added link right_sensor_middle_distal
- added link right_sensor_middle_proximal
- added link right_sensor_pinky_distal
- added link right_sensor_pinky_proximal
- added link right_sensor_ring_distal
- added link right_sensor_ring_proximal
- added link right_sensor_thumb_distal
- added link right_sensor_thumb_proximal
Joints:
- added joint right_sensor_dorsum_fixed: type fixed, parent R-Carpals_8d1f1041, child right_sensor_dorsum, origin xyz=0 0 0 rpy=1.57 0 0
- added joint right_sensor_index_distal_fixed: type fixed, parent I-FingerTipAssembly_ec49c16c, child right_sensor_index_distal, origin xyz=-0.004946 0.000001 0.045049 rpy=1.00 0 1.57
- added joint right_sensor_index_proximal_fixed: type fixed, parent I-PP_bacbd481, child right_sensor_index_proximal, origin xyz=0.00075 0 0.0185 rpy=1.00 0 1.57
- added joint right_sensor_middle_distal_fixed: type fixed, parent M-FingerTipAssembly_34afb748, child right_sensor_middle_distal, origin xyz=-0.004946 0.000001 0.045049 rpy=1.00 0 1.57
- added joint right_sensor_middle_proximal_fixed: type fixed, parent M-PP_08efa608, child right_sensor_middle_proximal, origin xyz=0.001 0 0.02 rpy=1.00 0 1.57
- added joint right_sensor_pinky_distal_fixed: type fixed, parent P-FingerTipAssembly_cd219176, child right_sensor_pinky_distal, origin xyz=-0.005452 0.000005 0.038056 rpy=1.00 0 1.57
- added joint right_sensor_pinky_proximal_fixed: type fixed, parent P-PP_1d411b9b, child right_sensor_pinky_proximal, origin xyz=0.0005 0 0.0155 rpy=1.00 0 1.57
- added joint right_sensor_ring_distal_fixed: type fixed, parent M-FingerTipAssembly_424a8e75, child right_sensor_ring_distal, origin xyz=-0.004946 0.000001 0.045049 rpy=1.00 0 1.57
- added joint right_sensor_ring_proximal_fixed: type fixed, parent M-PP_8660a1eb, child right_sensor_ring_proximal, origin xyz=0.001 0 0.02 rpy=1.00 0 1.57
- added joint right_sensor_thumb_distal_fixed: type fixed, parent T-DP_b7429e50, child right_sensor_thumb_distal, origin xyz=0.004104 -0.00019 0.030238 rpy=1.57 0 1.57
- added joint right_sensor_thumb_proximal_fixed: type fixed, parent T-PP_68395e98, child right_sensor_thumb_proximal, origin xyz=0.0005 0 0.016 rpy=1.57 0 1.57
